Commit message: Problem solved

File: turtlebot4_description/urdf/sensors/rplidar.urdf.xacro (robot description, xacro)
@@ -1,44 +1,64 @@
 <?xml version="1.0"?>
 <robot xmlns:xacro="http://ros.org/wiki/xacro">
-<xacro:macro name="rplidar" params="name parent_link gazebo *origin">
-  <xacro:include filename="$(find irobot_create_description)/urdf/common_properties.urdf.xacro"/>
-  <xacro:property name="mass"       value="0.17"/>
-  <xacro:property name="length_x"   value="${7.1*cm2m}" />
-  <xacro:property name="length_y"   value="${10*cm2m}" />
-  <xacro:property name="length_z"   value="${6*cm2m}" />
-  <xacro:property name="collision_x_offset"       value="${0*cm2m}" />
-  <xacro:property name="collision_y_offset"       value="${1.3*cm2m}" />
-  <xacro:property name="collision_z_offset"       value="${-1.9*cm2m}" />
-  <joint name="${name}_joint" type="fixed">
-    <parent link="${parent_link}"/>
-    <child link="${name}_link"/>
-    <xacro:insert_block name="origin"/>
-  </joint>
-  <link name="${name}_link">
-    <visual>
-      <geometry>
-        <mesh filename="package://turtlebot4_description/meshes/rplidar.dae" scale="1 1 1" />
-      </geometry>
-    </visual>
-    <collision>
-      <origin xyz="${collision_x_offset} ${collision_y_offset} ${collision_z_offset}"/>
-      <geometry>
-        <box size="${length_x} ${length_y} ${length_z}"/>
-      </geometry>
-    </collision>
-    <xacro:inertial_cuboid mass="0.17" x="${length_x}" y="${length_y}" z="${length_z}"/>
-  </link>
-  <gazebo reference="${name}_link">
-    <xacro:ray_sensor sensor_name="${name}" gazebo="${gazebo}"
-                  update_rate="62.0" visualize="1"
-                  h_samples="640" h_res="1.0" h_min_angle="${-pi}" h_max_angle="${pi}"
-                  r_min="0.164" r_max="12.0" r_res="0.01">
-                  <plugin name="dummy" filename="dummyfile"></plugin>
-    </xacro:ray_sensor>
-    <xacro:material_darkgray/>
-  </gazebo>
-  <gazebo reference="${name}_joint">
-    <preserveFixedJoint>true</preserveFixedJoint>
-  </gazebo>
-</xacro:macro>
+  <xacro:macro name="rplidar" params="name parent_link gazebo *origin">
+    <xacro:include filename="$(find irobot_create_description)/urdf/common_properties.urdf.xacro" />
+    <xacro:property name="mass" value="0.17" />
+    <xacro:property name="length_x" value="${7.1*cm2m}" />
+    <xacro:property name="length_y" value="${10*cm2m}" />
+    <xacro:property name="length_z" value="${6*cm2m}" />
+    <xacro:property name="collision_x_offset" value="${0*cm2m}" />
+    <xacro:property name="collision_y_offset" value="${1.3*cm2m}" />
+    <xacro:property name="collision_z_offset" value="${-1.9*cm2m}" />
+    <joint name="${name}_joint" type="fixed">
+      <parent link="${parent_link}" />
+      <child link="${name}_link" />
+      <xacro:insert_block name="origin" />
+    </joint>
+    <link name="${name}_link">
+      <visual>
+        <geometry>
+          <mesh filename="package://turtlebot4_description/meshes/rplidar.dae" scale="1 1 1" />
+        </geometry>
+      </visual>
+      <collision>
+        <origin xyz="${collision_x_offset} ${collision_y_offset} ${collision_z_offset}" />
+        <geometry>
+          <box size="${length_x} ${length_y} ${length_z}" />
+        </geometry>
+      </collision>
+      <xacro:inertial_cuboid mass="0.17" x="${length_x}" y="${length_y}" z="${length_z}" />
+    </link>
+    <gazebo reference="${name}_link">
+      <sensor name="${name}" type="gpu_lidar">
+        <always_on>true</always_on>
+        <visualize>true</visualize>
+        <update_rate>62.0</update_rate>
+        <lidar>
+          <scan>
+            <horizontal>
+              <samples>640</samples>
+              <resolution>1.0</resolution>
+              <min_angle>${-pi}</min_angle>
+              <max_angle>${pi}</max_angle>
+            </horizontal>
+            <vertical>
+              <samples>1</samples>
+              <resolution>1.0</resolution>
+              <min_angle>0.0</min_angle>
+              <max_angle>0.0</max_angle>
+            </vertical>
+          </scan>
+          <range>
+            <min>0.164</min>
+            <max>12.0</max>
+            <resolution>0.1</resolution>
+          </range>
+        </lidar>
+      </sensor>
+      <xacro:material_darkgray />
+    </gazebo>
+    <gazebo reference="${name}_joint">
+      <preserveFixedJoint>true</preserveFixedJoint>
+    </gazebo>
+  </xacro:macro>
 </robot>
